File: KC_NixieSupply5vTo170vMini/NixieSupply5vto170vDCMBoostMini.kicad_pcb (KiCad board)
At the start: 2 copper layers, 38.6 x 29 mm, 43 parts, among them J1 Screw_Terminal_1x02, J2 CONN_01X01, J3 CONN_01X01, J4 CONN_01X01, J5 CONN_01X01, J6 Screw_Terminal_1x03, P1 USB_OTG, Q1 FDS2672CT, Q26 MMBTA42, U1 UCC3803

Commit message: This saves Kicad version 4.0 o of the nixie power supplies.
Parts:
- moved G*** 0.91 mm to (151.3, 102.2)
Changed lines of the file:
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@@
-(kicad_pcb (version 4) (host pcbnew 4.0.6+dfsg1-1)
+(kicad_pcb (version 4) (host pcbnew 4.0.7-e2-6376~61~ubuntu18.04.1)
   (general
     (links 77)
@@
   (page A4)
   (layers
-    (0 F.Cu signal)
+    (0 F.Cu signal hide)
     (31 B.Cu signal)
     (34 B.Paste user)
@@
     (aux_axis_origin 136.0932 73.1774)
     (grid_origin 136.398 83.82)
-    (visible_elements 7FFEDE2B)
+    (visible_elements 7FFE9E2B)
     (pcbplotparams
       (layerselection 0x010f0_80000001)
@@
   )
   (module OSHW_logo_silkscreen-front_5mm (layer B.Cu)
-    (at 150.4315 102.2985 180)
+    (at 151.338 102.22 180)
     (fp_text reference G*** (at 0 -2.65176 180) (layer B.SilkS) hide
       (effects (font (size 0.22606 0.22606) (thickness 0.04318)) (justify mirror))

Commit message: The NewOrigin Zip file was used for the PCBWAY order This BOM was used for the PCBway order Updated the files to Rev 5 of Kicad
Parts:
- removed the G*** at (159.7, 108.5)
- removed the G*** at (151.3, 102.2)
- added G***: OSHW_logo_silkscreen-front_5mm, NixieSupply5vto170vDCMBoostMini_socket:OSHW_logo_silkscreen-front_5mm, B.Cu at (153.4, 102.5)
- added G***: LOGO, Symbol:copyright, B.Cu at (159.9, 108.2)
